Commit message: Changed mass and inertia values of baselink and fixed path issues for meshes

File: install/urdf_description/share/urdf_description/urdf/URDF.xacro (robot description, xacro)
@@ -7,6 +7,6 @@
   <inertial>
     <origin xyz="0.0 0.0 0.0" rpy="0 0 0"/>
-    <mass value="0.0"/>
-    <inertia ixx="0.0" iyy="0.0" izz="0.0" ixy="0.0" iyz="0.0" ixz="0.0"/>
+    <mass value="50.0"/> <!-- Base link mass test value-->
+    <inertia ixx="1.5" iyy="2.5" izz="3.5" ixy="0.0" iyz="0.0" ixz="0.0"/> <!-- Base link inertia test values-->
   </inertial>
   <visual>

Commit message: Safely restored all project files

File: install/urdf_description/share/urdf_description/urdf/URDF.xacro (robot description, xacro)
@@ -6,4 +6,5 @@
 <link name="base_link">
   <inertial>
+<<<<<<< HEAD
     <origin xyz="0 0 0" rpy="0 0 0"/>
     <mass value="50.0"/>
@@ -12,4 +13,12 @@
   <visual>
     <origin xyz="0 0 0" rpy="0 0 0"/>
+=======
+    <origin xyz="0.0 0.0 0.0" rpy="0 0 0"/>
+    <mass value="50.0"/> <!-- Base link mass test value-->
+    <inertia ixx="1.5" iyy="2.5" izz="3.5" ixy="0.0" iyz="0.0" ixz="0.0"/> <!-- Base link inertia test values-->
+  </inertial>
+  <visual>
+    <origin xyz="0 0 0" rpy="0 0 0"/>
+>>>>>>> caddd7ff5a319ac415dbe87685f8ec4c434882f2
     <geometry>
       <mesh filename="package://urdf_description/meshes/base_link.stl" scale="0.001 0.001 0.001"/>
@@ -17,4 +26,7 @@
     <material name="silver"/>
   </visual>
+<<<<<<< HEAD
+=======
+>>>>>>> caddd7ff5a319ac415dbe87685f8ec4c434882f2
   <collision>
     <origin xyz="0 0 0" rpy="0 0 0"/>
@@ -24,4 +36,15 @@
   </collision>
 </link>
+<<<<<<< HEAD
+=======
+<!-- BASE_FOOTPRINT LINK -->
+<joint name="base_footprint_joint" type="fixed">
+    <parent link="base_link"/>
+    <child link="base_footprint"/>
+    <origin xyz="0 0 0" rpy="0 0 0"/>
+</joint>
+<link name="base_footprint">
+</link>
+>>>>>>> caddd7ff5a319ac415dbe87685f8ec4c434882f2
 <link name="Bogie2_1">
   <inertial>
@@ -84,4 +107,5 @@
   </collision>
 </link>
+<<<<<<< HEAD
 <link name="Bar1_1_sph_x">
   <inertial>
@@ -126,4 +150,6 @@
   </inertial>
 </link>
+=======
+>>>>>>> caddd7ff5a319ac415dbe87685f8ec4c434882f2
 <link name="Bar1_2">
   <inertial>
@@ -166,4 +192,5 @@
   </collision>
 </link>
+<<<<<<< HEAD
 <link name="Bar2_1_sph_x">
   <inertial>
@@ -187,4 +214,6 @@
   </inertial>
 </link>
+=======
+>>>>>>> caddd7ff5a319ac415dbe87685f8ec4c434882f2
 <link name="Bar2_2">
   <inertial>
@@ -207,4 +236,5 @@
   </collision>
 </link>
+<<<<<<< HEAD
 <link name="Bar2_2_sph_x">
   <inertial>
@@ -228,4 +258,6 @@
   </inertial>
 </link>
+=======
+>>>>>>> caddd7ff5a319ac415dbe87685f8ec4c434882f2
 <link name="Wheel1_1">
   <inertial>
@@ -408,9 +440,14 @@
   </collision>
 </link>
+<<<<<<< HEAD
 <joint name="Revolute_4" type="continuous">
+=======
+<joint name="Revolute 4" type="continuous">
+>>>>>>> caddd7ff5a319ac415dbe87685f8ec4c434882f2
   <origin xyz="0.103766 -0.219571 -0.0607" rpy="0 0 0"/>
   <parent link="Bogie1_1"/>
   <child link="Bogie2_1"/>
   <axis xyz="-0.708966 -0.677955 0.194277"/>
+<<<<<<< HEAD
   <dynamics damping="3.0" friction="0.2"/>
 </joint>
@@ -448,12 +485,45 @@
 <!-- Diff1 pivot on base — passive revolute, NOT continuous -->
 <joint name="Revolute_5" type="revolute">
+=======
+</joint>
+<joint name="Revolute 5" type="continuous">
+>>>>>>> caddd7ff5a319ac415dbe87685f8ec4c434882f2
   <origin xyz="0.342141 -0.375854 0.3869" rpy="0 0 0"/>
   <parent link="base_link"/>
   <child link="Diff1_1"/>
   <axis xyz="0.626432 -0.731916 -0.268109"/>
+<<<<<<< HEAD
   <limit lower="-0.5" upper="0.5" effort="0" velocity="1"/>
   <dynamics damping="3.0" friction="1.0"/>
 </joint>
 <joint name="Revolute_10" type="continuous">
+=======
+</joint>
+<joint name="Revolute 6" type="continuous">
+  <origin xyz="0.186039 -0.110927 0.194654" rpy="0 0 0"/>
+  <parent link="Bogie3_1"/>
+  <child link="Bar1_1"/>
+  <axis xyz="0.699606 -0.64133 0.315035"/>
+</joint>
+<joint name="Revolute 7" type="continuous">
+  <origin xyz="0.236664 0.188148 -0.011824" rpy="0 0 0"/>
+  <parent link="Diff1_1"/>
+  <child link="Bar1_2"/>
+  <axis xyz="0.626432 -0.731916 -0.268109"/>
+</joint>
+<joint name="Revolute 8" type="continuous">
+  <origin xyz="0.125165 -0.12932 0.102633" rpy="0 0 0"/>
+  <parent link="Bogie1_1"/>
+  <child link="Bar2_1"/>
+  <axis xyz="0.005692 -0.280968 -0.9597"/>
+</joint>
+<joint name="Revolute 9" type="continuous">
+  <origin xyz="-0.21948 -0.208225 0.00447" rpy="0 0 0"/>
+  <parent link="Diff1_1"/>
+  <child link="Bar2_2"/>
+  <axis xyz="0.626432 -0.731916 -0.268109"/>
+</joint>
+<joint name="Revolute 10" type="continuous">
+>>>>>>> caddd7ff5a319ac415dbe87685f8ec4c434882f2
   <origin xyz="-0.323557 0.444523 0.206988" rpy="0 0 0"/>
   <parent link="Bogie3_1"/>
@@ -461,5 +531,9 @@
   <axis xyz="-0.708966 -0.677955 0.194277"/>
 </joint>
+<<<<<<< HEAD
 <joint name="Revolute_11" type="continuous">
+=======
+<joint name="Revolute 11" type="continuous">
+>>>>>>> caddd7ff5a319ac415dbe87685f8ec4c434882f2
   <origin xyz="-0.141623 0.254762 0.208719" rpy="0 0 0"/>
   <parent link="Bogie4_1"/>
@@ -467,5 +541,9 @@
   <axis xyz="0.708966 0.677955 -0.194277"/>
 </joint>
+<<<<<<< HEAD
 <joint name="Revolute_12" type="continuous">
+=======
+<joint name="Revolute 12" type="continuous">
+>>>>>>> caddd7ff5a319ac415dbe87685f8ec4c434882f2
   <origin xyz="-0.228777 0.257791 -0.098632" rpy="0 0 0"/>
   <parent link="Bogie4_1"/>
@@ -473,5 +551,9 @@
   <axis xyz="0.708966 0.677955 -0.194277"/>
 </joint>
+<<<<<<< HEAD
 <joint name="Revolute_13" type="continuous">
+=======
+<joint name="Revolute 13" type="continuous">
+>>>>>>> caddd7ff5a319ac415dbe87685f8ec4c434882f2
   <origin xyz="-0.288513 0.111749 -0.499405" rpy="0 0 0"/>
   <parent link="Bogie1_1"/>
@@ -479,5 +561,9 @@
   <axis xyz="-0.708966 -0.677955 0.194277"/>
 </joint>
+<<<<<<< HEAD
 <joint name="Revolute_14" type="continuous">
+=======
+<joint name="Revolute 14" type="continuous">
+>>>>>>> caddd7ff5a319ac415dbe87685f8ec4c434882f2
   <origin xyz="0.174314 -0.273113 -0.153456" rpy="0 0 0"/>
   <parent link="Bogie2_1"/>
@@ -485,5 +571,9 @@
   <axis xyz="0.708966 0.677955 -0.194277"/>
 </joint>
+<<<<<<< HEAD
 <joint name="Revolute_15" type="continuous">
+=======
+<joint name="Revolute 15" type="continuous">
+>>>>>>> caddd7ff5a319ac415dbe87685f8ec4c434882f2
   <origin xyz="0.221257 -0.232364 0.159922" rpy="0 0 0"/>
   <parent link="Bogie2_1"/>
@@ -491,39 +581,67 @@
   <axis xyz="0.708966 0.677955 -0.194277"/>
 </joint>
+<<<<<<< HEAD
 <joint name="Revolute_1" type="continuous">
+=======
+<joint name="Revolute 1" type="continuous">
+>>>>>>> caddd7ff5a319ac415dbe87685f8ec4c434882f2
   <origin xyz="-0.020622 0.044907 -0.245401" rpy="0 0 0"/>
   <parent link="Bogie3_1"/>
   <child link="Bogie4_1"/>
   <axis xyz="0.708966 0.677955 -0.194277"/>
+<<<<<<< HEAD
   <dynamics damping="3.0" friction="0.2"/>
 </joint>
 <joint name="Revolute_17" type="revolute">
+=======
+</joint>
+<joint name="Revolute 17" type="continuous">
+>>>>>>> caddd7ff5a319ac415dbe87685f8ec4c434882f2
   <origin xyz="0.392766 -0.076779 0.180422" rpy="0 0 0"/>
   <parent link="base_link"/>
   <child link="Bogie3_1"/>
   <axis xyz="0.708966 0.677955 -0.194277"/>
+<<<<<<< HEAD
   <limit lower = "-0.5" upper = "0.5" effort = "0" veolcity = "1"/>
   <dynamics damping="3.0" friction="0.2"/>
 </joint>
 <joint name="Revolute_18" type="revolute">
+=======
+</joint>
+<joint name="Revolute 18" type="continuous">
+>>>>>>> caddd7ff5a319ac415dbe87685f8ec4c434882f2
   <origin xyz="-0.002504 -0.454759 0.288737" rpy="0 0 0"/>
   <parent link="base_link"/>
   <child link="Bogie1_1"/>
   <axis xyz="0.708966 0.677955 -0.194277"/>
+<<<<<<< HEAD
   <limit lower = "-0.5" upper = "0.5" effort = "0" veolcity = "1"/>
   <dynamics damping="3.0" friction="0.2"/>
+=======
+>>>>>>> caddd7ff5a319ac415dbe87685f8ec4c434882f2
 </joint>
 <ros2_control name="IgnitionSystem" type="system">
+<<<<<<< HEAD
+=======
+>>>>>>> caddd7ff5a319ac415dbe87685f8ec4c434882f2
   <hardware>
     <plugin>ign_ros2_control/IgnitionSystem</plugin>
   </hardware>
+<<<<<<< HEAD
   <joint name="Revolute_10">
     <command_interface name="velocity">
       <param name="min">-10.0</param>
       <param name="max">10.0</param>
+=======
+  <joint name="Revolute 10">
+    <command_interface name="velocity">
+      <param name="min">-10</param>
+      <param name="max">10</param>
+>>>>>>> caddd7ff5a319ac415dbe87685f8ec4c434882f2
     </command_interface>
     <state_interface name="position"/>
     <state_interface name="velocity"/>
   </joint>
+<<<<<<< HEAD
   <joint name="Revolute_11">
     <command_interface name="velocity">
@@ -576,4 +694,27 @@
   <origin xyz="0.25 0 0.35" rpy="0 0 0"/>
 </joint>
+=======
+  <joint name="Revolute 11">
+    <command_interface name="velocity"><param name="min">-10</param><param name="max">10</param></command_interface>
+    <state_interface name="position"/><state_interface name="velocity"/>
+  </joint>
+  <joint name="Revolute 12">
+    <command_interface name="velocity"/>
+    <state_interface name="position"/><state_interface name="velocity"/>
+  </joint>
+  <joint name="Revolute 13">
+    <command_interface name="velocity"/>
+    <state_interface name="position"/><state_interface name="velocity"/>
+  </joint>
+  <joint name="Revolute 14">
+    <command_interface name="velocity"/>
+    <state_interface name="position"/><state_interface name="velocity"/>
+  </joint>
+  <joint name="Revolute 15">
+    <command_interface name="velocity"/>
+    <state_interface name="position"/><state_interface name="velocity"/>
+  </joint>
+</ros2_control>
+>>>>>>> caddd7ff5a319ac415dbe87685f8ec4c434882f2
 <!-- Add before the closing </robot> tag -->
 <link name="lidar_link">

File: urdf/URDF.xacro (robot description, xacro)
@@ -6,4 +6,5 @@
 <link name="base_link">
   <inertial>
+<<<<<<< HEAD
     <origin xyz="0 0 0" rpy="0 0 0"/>
     <mass value="50.0"/>
@@ -12,4 +13,12 @@
   <visual>
     <origin xyz="0 0 0" rpy="0 0 0"/>
+=======
+    <origin xyz="0.0 0.0 0.0" rpy="0 0 0"/>
+    <mass value="50.0"/> <!-- Base link mass test value-->
+    <inertia ixx="1.5" iyy="2.5" izz="3.5" ixy="0.0" iyz="0.0" ixz="0.0"/> <!-- Base link inertia test values-->
+  </inertial>
+  <visual>
+    <origin xyz="0 0 0" rpy="0 0 0"/>
+>>>>>>> caddd7ff5a319ac415dbe87685f8ec4c434882f2
     <geometry>
       <mesh filename="package://urdf_description/meshes/base_link.stl" scale="0.001 0.001 0.001"/>
@@ -17,4 +26,7 @@
     <material name="silver"/>
   </visual>
+<<<<<<< HEAD
+=======
+>>>>>>> caddd7ff5a319ac415dbe87685f8ec4c434882f2
   <collision>
     <origin xyz="0 0 0" rpy="0 0 0"/>
@@ -24,4 +36,15 @@
   </collision>
 </link>
+<<<<<<< HEAD
+=======
+<!-- BASE_FOOTPRINT LINK -->
+<joint name="base_footprint_joint" type="fixed">
+    <parent link="base_link"/>
+    <child link="base_footprint"/>
+    <origin xyz="0 0 0" rpy="0 0 0"/>
+</joint>
+<link name="base_footprint">
+</link>
+>>>>>>> caddd7ff5a319ac415dbe87685f8ec4c434882f2
 <link name="Bogie2_1">
   <inertial>
@@ -84,4 +107,5 @@
   </collision>
 </link>
+<<<<<<< HEAD
 <link name="Bar1_1_sph_x">
   <inertial>
@@ -126,4 +150,6 @@
   </inertial>
 </link>
+=======
+>>>>>>> caddd7ff5a319ac415dbe87685f8ec4c434882f2
 <link name="Bar1_2">
   <inertial>
@@ -166,4 +192,5 @@
   </collision>
 </link>
+<<<<<<< HEAD
 <link name="Bar2_1_sph_x">
   <inertial>
@@ -187,4 +214,6 @@
   </inertial>
 </link>
+=======
+>>>>>>> caddd7ff5a319ac415dbe87685f8ec4c434882f2
 <link name="Bar2_2">
   <inertial>
@@ -207,4 +236,5 @@
   </collision>
 </link>
+<<<<<<< HEAD
 <link name="Bar2_2_sph_x">
   <inertial>
@@ -228,4 +258,6 @@
   </inertial>
 </link>
+=======
+>>>>>>> caddd7ff5a319ac415dbe87685f8ec4c434882f2
 <link name="Wheel1_1">
   <inertial>
@@ -408,16 +440,26 @@
   </collision>
 </link>
+<<<<<<< HEAD
 <joint name="Revolute_4" type="continuous">
+=======
+<joint name="Revolute 4" type="continuous">
+>>>>>>> caddd7ff5a319ac415dbe87685f8ec4c434882f2
   <origin xyz="0.103766 -0.219571 -0.0607" rpy="0 0 0"/>
   <parent link="Bogie1_1"/>
   <child link="Bogie2_1"/>
   <axis xyz="-0.708966 -0.677955 0.194277"/>
+<<<<<<< HEAD
   <dynamics damping="3.0" friction="0.2"/>
 </joint>
 <joint name="Revolute_5" type="continuous">
+=======
+</joint>
+<joint name="Revolute 5" type="continuous">
+>>>>>>> caddd7ff5a319ac415dbe87685f8ec4c434882f2
   <origin xyz="0.342141 -0.375854 0.3869" rpy="0 0 0"/>
   <parent link="base_link"/>
   <child link="Diff1_1"/>
   <axis xyz="0.626432 -0.731916 -0.268109"/>
+<<<<<<< HEAD
   <dynamics damping="3.0" friction="0.2"/>
 </joint>
@@ -515,4 +557,32 @@
 </joint>
 <joint name="Revolute_10" type="continuous">
+=======
+</joint>
+<joint name="Revolute 6" type="continuous">
+  <origin xyz="0.186039 -0.110927 0.194654" rpy="0 0 0"/>
+  <parent link="Bogie3_1"/>
+  <child link="Bar1_1"/>
+  <axis xyz="0.699606 -0.64133 0.315035"/>
+</joint>
+<joint name="Revolute 7" type="continuous">
+  <origin xyz="0.236664 0.188148 -0.011824" rpy="0 0 0"/>
+  <parent link="Diff1_1"/>
+  <child link="Bar1_2"/>
+  <axis xyz="0.626432 -0.731916 -0.268109"/>
+</joint>
+<joint name="Revolute 8" type="continuous">
+  <origin xyz="0.125165 -0.12932 0.102633" rpy="0 0 0"/>
+  <parent link="Bogie1_1"/>
+  <child link="Bar2_1"/>
+  <axis xyz="0.005692 -0.280968 -0.9597"/>
+</joint>
+<joint name="Revolute 9" type="continuous">
+  <origin xyz="-0.21948 -0.208225 0.00447" rpy="0 0 0"/>
+  <parent link="Diff1_1"/>
+  <child link="Bar2_2"/>
+  <axis xyz="0.626432 -0.731916 -0.268109"/>
+</joint>
+<joint name="Revolute 10" type="continuous">
+>>>>>>> caddd7ff5a319ac415dbe87685f8ec4c434882f2
   <origin xyz="-0.323557 0.444523 0.206988" rpy="0 0 0"/>
   <parent link="Bogie3_1"/>
@@ -520,5 +590,9 @@
   <axis xyz="-0.708966 -0.677955 0.194277"/>
 </joint>
+<<<<<<< HEAD
 <joint name="Revolute_11" type="continuous">
+=======
+<joint name="Revolute 11" type="continuous">
+>>>>>>> caddd7ff5a319ac415dbe87685f8ec4c434882f2
   <origin xyz="-0.141623 0.254762 0.208719" rpy="0 0 0"/>
   <parent link="Bogie4_1"/>
@@ -526,5 +600,9 @@
   <axis xyz="0.708966 0.677955 -0.194277"/>
 </joint>
+<<<<<<< HEAD
 <joint name="Revolute_12" type="continuous">
+=======
+<joint name="Revolute 12" type="continuous">
+>>>>>>> caddd7ff5a319ac415dbe87685f8ec4c434882f2
   <origin xyz="-0.228777 0.257791 -0.098632" rpy="0 0 0"/>
   <parent link="Bogie4_1"/>
@@ -532,5 +610,9 @@
   <axis xyz="0.708966 0.677955 -0.194277"/>
 </joint>
+<<<<<<< HEAD
 <joint name="Revolute_13" type="continuous">
+=======
+<joint name="Revolute 13" type="continuous">
+>>>>>>> caddd7ff5a319ac415dbe87685f8ec4c434882f2
   <origin xyz="-0.288513 0.111749 -0.499405" rpy="0 0 0"/>
   <parent link="Bogie1_1"/>
@@ -538,5 +620,9 @@
   <axis xyz="-0.708966 -0.677955 0.194277"/>
 </joint>
+<<<<<<< HEAD
 <joint name="Revolute_14" type="continuous">
+=======
+<joint name="Revolute 14" type="continuous">
+>>>>>>> caddd7ff5a319ac415dbe87685f8ec4c434882f2
   <origin xyz="0.174314 -0.273113 -0.153456" rpy="0 0 0"/>
   <parent link="Bogie2_1"/>
@@ -544,5 +630,9 @@
   <axis xyz="0.708966 0.677955 -0.194277"/>
 </joint>
+<<<<<<< HEAD
 <joint name="Revolute_15" type="continuous">
+=======
+<joint name="Revolute 15" type="continuous">
+>>>>>>> caddd7ff5a319ac415dbe87685f8ec4c434882f2
   <origin xyz="0.221257 -0.232364 0.159922" rpy="0 0 0"/>
   <parent link="Bogie2_1"/>
@@ -550,37 +640,65 @@
   <axis xyz="0.708966 0.677955 -0.194277"/>
 </joint>
+<<<<<<< HEAD
 <joint name="Revolute_1" type="continuous">
+=======
+<joint name="Revolute 1" type="continuous">
+>>>>>>> caddd7ff5a319ac415dbe87685f8ec4c434882f2
   <origin xyz="-0.020622 0.044907 -0.245401" rpy="0 0 0"/>
   <parent link="Bogie3_1"/>
   <child link="Bogie4_1"/>
   <axis xyz="0.708966 0.677955 -0.194277"/>
+<<<<<<< HEAD
   <dynamics damping="3.0" friction="0.2"/>
 </joint>
 <joint name="Revolute_17" type="continuous">
+=======
+</joint>
+<joint name="Revolute 17" type="continuous">
+>>>>>>> caddd7ff5a319ac415dbe87685f8ec4c434882f2
   <origin xyz="0.392766 -0.076779 0.180422" rpy="0 0 0"/>
   <parent link="base_link"/>
   <child link="Bogie3_1"/>
   <axis xyz="0.708966 0.677955 -0.194277"/>
+<<<<<<< HEAD
   <dynamics damping="3.0" friction="0.2"/>
 </joint>
 <joint name="Revolute_18" type="continuous">
+=======
+</joint>
+<joint name="Revolute 18" type="continuous">
+>>>>>>> caddd7ff5a319ac415dbe87685f8ec4c434882f2
   <origin xyz="-0.002504 -0.454759 0.288737" rpy="0 0 0"/>
   <parent link="base_link"/>
   <child link="Bogie1_1"/>
   <axis xyz="0.708966 0.677955 -0.194277"/>
+<<<<<<< HEAD
   <dynamics damping="3.0" friction="0.2"/>
+=======
+>>>>>>> caddd7ff5a319ac415dbe87685f8ec4c434882f2
 </joint>
 <ros2_control name="IgnitionSystem" type="system">
+<<<<<<< HEAD
+=======
+>>>>>>> caddd7ff5a319ac415dbe87685f8ec4c434882f2
   <hardware>
     <plugin>ign_ros2_control/IgnitionSystem</plugin>
   </hardware>
+<<<<<<< HEAD
   <joint name="Revolute_10">
     <command_interface name="velocity">
       <param name="min">-10.0</param>
       <param name="max">10.0</param>
+=======
+  <joint name="Revolute 10">
+    <command_interface name="velocity">
+      <param name="min">-10</param>
+      <param name="max">10</param>
+>>>>>>> caddd7ff5a319ac415dbe87685f8ec4c434882f2
     </command_interface>
     <state_interface name="position"/>
     <state_interface name="velocity"/>
   </joint>
+<<<<<<< HEAD
   <joint name="Revolute_11">
     <command_interface name="velocity">
@@ -633,4 +751,27 @@
   <origin xyz="0.25 0 0.35" rpy="0 0 0"/>
 </joint>
+=======
+  <joint name="Revolute 11">
+    <command_interface name="velocity"><param name="min">-10</param><param name="max">10</param></command_interface>
+    <state_interface name="position"/><state_interface name="velocity"/>
+  </joint>
+  <joint name="Revolute 12">
+    <command_interface name="velocity"/>
+    <state_interface name="position"/><state_interface name="velocity"/>
+  </joint>
+  <joint name="Revolute 13">
+    <command_interface name="velocity"/>
+    <state_interface name="position"/><state_interface name="velocity"/>
+  </joint>
+  <joint name="Revolute 14">
+    <command_interface name="velocity"/>
+    <state_interface name="position"/><state_interface name="velocity"/>
+  </joint>
+  <joint name="Revolute 15">
+    <command_interface name="velocity"/>
+    <state_interface name="position"/><state_interface name="velocity"/>
+  </joint>
+</ros2_control>
+>>>>>>> caddd7ff5a319ac415dbe87685f8ec4c434882f2
 <!-- Add before the closing </robot> tag -->
 <link name="lidar_link">
