Commit message: Replace URDF with clean simplified rocker-bogie design
- Removed all merge conflicts
- Removed orphaned Bar and Diff1 links
- Removed redundant spherical joint chains  
- Clean rocker-bogie structure with differential bar
- 4 articulation points: front rocker, center boom, rear rocker, diff bar connection
- All 6 wheels properly controlled
- Removed outdated URDF.trans include

File: urdf/URDF.xacro (robot description, xacro)
@@ -2,9 +2,8 @@
 <robot name="URDF" xmlns:xacro="http://www.ros.org/wiki/xacro">
 <xacro:include filename="$(find urdf_description)/urdf/materials.xacro"/>
-<xacro:include filename="$(find urdf_description)/urdf/URDF.trans" />
 <xacro:include filename="$(find urdf_description)/urdf/URDF.gazebo" />
+<!-- BASE LINK (Chassis) -->
 <link name="base_link">
   <inertial>
-<<<<<<< HEAD
     <origin xyz="0 0 0" rpy="0 0 0"/>
     <mass value="50.0"/>
@@ -13,12 +12,4 @@
   <visual>
     <origin xyz="0 0 0" rpy="0 0 0"/>
-=======
-    <origin xyz="0.0 0.0 0.0" rpy="0 0 0"/>
-    <mass value="50.0"/> <!-- Base link mass test value-->
-    <inertia ixx="1.5" iyy="2.5" izz="3.5" ixy="0.0" iyz="0.0" ixz="0.0"/> <!-- Base link inertia test values-->
-  </inertial>
-  <visual>
-    <origin xyz="0 0 0" rpy="0 0 0"/>
->>>>>>> caddd7ff5a319ac415dbe87685f8ec4c434882f2
     <geometry>
       <mesh filename="package://urdf_description/meshes/base_link.stl" scale="0.001 0.001 0.001"/>
@@ -26,7 +17,4 @@
     <material name="silver"/>
   </visual>
-<<<<<<< HEAD
-=======
->>>>>>> caddd7ff5a319ac415dbe87685f8ec4c434882f2
   <collision>
     <origin xyz="0 0 0" rpy="0 0 0"/>
@@ -36,16 +24,48 @@
   </collision>
 </link>
-<<<<<<< HEAD
-=======
-<!-- BASE_FOOTPRINT LINK -->
-<joint name="base_footprint_joint" type="fixed">
-    <parent link="base_link"/>
-    <child link="base_footprint"/>
-    <origin xyz="0 0 0" rpy="0 0 0"/>
-</joint>
-<link name="base_footprint">
-</link>
->>>>>>> caddd7ff5a319ac415dbe87685f8ec4c434882f2
-<link name="Bogie2_1">
+<!-- FRONT ROCKER ARM (Bogie3_1) -->
+<link name="bogie_front">
+  <inertial>
+    <origin xyz="-0.24598384655946126 0.3733777171361519 0.23572313584798862" rpy="0 0 0"/>
+    <mass value="2.7421522792750093"/>
+    <inertia ixx="0.017885" iyy="0.018532" izz="0.031298" ixy="0.00644" iyz="0.004516" ixz="-0.002275"/>
+  </inertial>
+  <visual>
+    <origin xyz="-0.392766 0.076779 -0.180422" rpy="0 0 0"/>
+    <geometry>
+      <mesh filename="package://urdf_description/meshes/Bogie3_1.stl" scale="0.001 0.001 0.001"/>
+    </geometry>
+    <material name="silver"/>
+  </visual>
+  <collision>
+    <origin xyz="-0.392766 0.076779 -0.180422" rpy="0 0 0"/>
+    <geometry>
+      <mesh filename="package://urdf_description/meshes/Bogie3_1.stl" scale="0.001 0.001 0.001"/>
+    </geometry>
+  </collision>
+</link>
+<!-- FRONT WHEEL (on Front Rocker) -->
+<link name="wheel_front">
+  <inertial>
+    <origin xyz="0 0 0" rpy="0 0 0"/>
+    <mass value="18.64386375159242"/>
+    <inertia ixx="0.207999" iyy="0.203936" izz="0.164115" ixy="0.045369" iyz="-0.012432" ixz="-0.013001"/>
+  </inertial>
+  <visual>
+    <origin xyz="-0.323557 0.444523 0.206988" rpy="0 0 0"/>
+    <geometry>
+      <mesh filename="package://urdf_description/meshes/Wheel1_1.stl" scale="0.001 0.001 0.001"/>
+    </geometry>
+    <material name="silver"/>
+  </visual>
+  <collision>
+    <origin xyz="-0.323557 0.444523 0.206988" rpy="0 0 0"/>
+    <geometry>
+      <mesh filename="package://urdf_description/meshes/Wheel1_1.stl" scale="0.001 0.001 0.001"/>
+    </geometry>
+  </collision>
+</link>
+<!-- CENTER BOGIE (Differential Bar System - Bogie2_1) -->
+<link name="bogie_center">
   <inertial>
     <origin xyz="0.06251976698493288 -0.11015246561255954 0.004955724047181781" rpy="0 0 0"/>
@@ -67,244 +87,32 @@
   </collision>
 </link>
-<link name="Diff1_1">
-  <inertial>
-    <origin xyz="0.008076545764013954 -0.009489204709679455 -0.003466898798053508" rpy="0 0 0"/>
-    <mass value="1.4810144679840673"/>
-    <inertia ixx="0.027522" iyy="0.036276" izz="0.063269" ixy="-0.031063" iyz="0.0011" ixz="0.001287"/>
-  </inertial>
-  <visual>
-    <origin xyz="-0.342141 0.375854 -0.3869" rpy="0 0 0"/>
-    <geometry>
-      <mesh filename="package://urdf_description/meshes/Diff1_1.stl" scale="0.001 0.001 0.001"/>
-    </geometry>
-    <material name="silver"/>
-  </visual>
-  <collision>
-    <origin xyz="-0.342141 0.375854 -0.3869" rpy="0 0 0"/>
-    <geometry>
-      <mesh filename="package://urdf_description/meshes/Diff1_1.stl" scale="0.001 0.001 0.001"/>
-    </geometry>
-  </collision>
-</link>
-<link name="Bar1_1">
-  <inertial>
-    <origin xyz="0.045351822773323336 -0.032846199265664 0.0840140470710965" rpy="0 0 0"/>
-    <mass value="0.28218703834108916"/>
-    <inertia ixx="0.001138" iyy="0.001274" izz="0.000443" ixy="0.000207" iyz="0.000383" ixz="-0.000529"/>
-  </inertial>
-  <visual>
-    <origin xyz="-0.488102 0.122014 -0.207048" rpy="0 0 0"/>
-    <geometry>
-      <mesh filename="package://urdf_description/meshes/Bar1_1.stl" scale="0.001 0.001 0.001"/>
-    </geometry>
-    <material name="silver"/>
-  </visual>
-  <collision>
-    <origin xyz="-0.488102 0.122014 -0.207048" rpy="0 0 0"/>
-    <geometry>
-      <mesh filename="package://urdf_description/meshes/Bar1_1.stl" scale="0.001 0.001 0.001"/>
-    </geometry>
-  </collision>
-</link>
-<<<<<<< HEAD
-<link name="Bar1_1_sph_x">
-  <inertial>
-    <mass value="0.001"/>
-    <inertia ixx="1e-6" iyy="1e-6" izz="1e-6"
-             ixy="0" iyz="0" ixz="0"/>
-  </inertial>
-</link>
-<link name="Bar1_1_sph_y">
-  <inertial>
-    <mass value="0.001"/>
-    <inertia ixx="1e-6" iyy="1e-6" izz="1e-6"
-             ixy="0" iyz="0" ixz="0"/>
-  </inertial>
-</link>
-<link name="Bar1_1_sph_z">
-  <inertial>
-    <mass value="0.001"/>
-    <inertia ixx="1e-6" iyy="1e-6" izz="1e-6"
-             ixy="0" iyz="0" ixz="0"/>
-  </inertial>
-</link>
-<link name="Bar1_2_sph_x">
-  <inertial>
-  <mass value="0.001"/>
-    <inertia ixx="1e-6" iyy="1e-6" izz="1e-6"
-             ixy="0" iyz="0" ixz="0"/>
-  </inertial>
-</link>
-<link name="Bar1_2_sph_y">
-  <inertial>
-    <mass value="0.001"/>
-    <inertia ixx="1e-6" iyy="1e-6" izz="1e-6"
-             ixy="0" iyz="0" ixz="0"/>
-  </inertial>
-</link>
-<link name="Bar1_2_sph_z">
-  <inertial>
-    <mass value="0.001"/>
-    <inertia ixx="1e-6" iyy="1e-6" izz="1e-6"
-             ixy="0" iyz="0" ixz="0"/>
-  </inertial>
-</link>
-=======
->>>>>>> caddd7ff5a319ac415dbe87685f8ec4c434882f2
-<link name="Bar1_2">
-  <inertial>
-    <origin xyz="-0.0453511772266767 0.03284580073433602 -0.08401395292890351" rpy="0 0 0"/>
-    <mass value="0.28218703834108916"/>
-    <inertia ixx="0.001138" iyy="0.001274" izz="0.000443" ixy="0.000207" iyz="0.000383" ixz="-0.000529"/>
-  </inertial>
-  <visual>
-    <origin xyz="-0.578805 0.187706 -0.375076" rpy="0 0 0"/>
-    <geometry>
-      <mesh filename="package://urdf_description/meshes/Bar1_1.stl" scale="0.001 0.001 0.001"/>
-    </geometry>
-    <material name="silver"/>
-  </visual>
-  <collision>
-    <origin xyz="-0.578805 0.187706 -0.375076" rpy="0 0 0"/>
-    <geometry>
-      <mesh filename="package://urdf_description/meshes/Bar1_1.stl" scale="0.001 0.001 0.001"/>
-    </geometry>
-  </collision>
-</link>
-<link name="Bar2_1">
-  <inertial>
-    <origin xyz="0.07413351250862066 -0.06852176424171452 -0.001718250267395638" rpy="0 0 0"/>
-    <mass value="0.28218703834108916"/>
-    <inertia ixx="0.00066" iyy="0.000771" izz="0.001423" ixy="0.000705" iyz="-1.6e-05" ixz="1.8e-05"/>
-  </inertial>
-  <visual>
-    <origin xyz="0.025606 0.447036 -0.394807" rpy="0 0 0"/>
-    <geometry>
-      <mesh filename="package://urdf_description/meshes/Bar2_1.stl" scale="0.001 0.001 0.001"/>
-    </geometry>
-    <material name="silver"/>
-  </visual>
-  <collision>
-    <origin xyz="0.025606 0.447036 -0.394807" rpy="0 0 0"/>
-    <geometry>
-      <mesh filename="package://urdf_description/meshes/Bar2_1.stl" scale="0.001 0.001 0.001"/>
-    </geometry>
-  </collision>
-</link>
-<<<<<<< HEAD
-<link name="Bar2_1_sph_x">
-  <inertial>
-  <mass value="0.001"/>
-    <inertia ixx="1e-6" iyy="1e-6" izz="1e-6"
-             ixy="0" iyz="0" ixz="0"/>
-  </inertial>
-</link>
-<link name="Bar2_1_sph_y">
-  <inertial>
-    <mass value="0.001"/>
-    <inertia ixx="1e-6" iyy="1e-6" izz="1e-6"
-             ixy="0" iyz="0" ixz="0"/>
-  </inertial>
-</link>
-<link name="Bar2_1_sph_z">
-  <inertial>
-    <mass value="0.001"/>
-    <inertia ixx="1e-6" iyy="1e-6" izz="1e-6"
-             ixy="0" iyz="0" ixz="0"/>
-  </inertial>
-</link>
-=======
->>>>>>> caddd7ff5a319ac415dbe87685f8ec4c434882f2
-<link name="Bar2_2">
-  <inertial>
-    <origin xyz="-0.07413348749137935 0.0685212357582855 0.0017187497326043855" rpy="0 0 0"/>
-    <mass value="0.28218703834108916"/>
-    <inertia ixx="0.00066" iyy="0.000771" izz="0.001423" ixy="0.000705" iyz="-1.6e-05" ixz="1.8e-05"/>
-  </inertial>
-  <visual>
-    <origin xyz="-0.122661 0.584079 -0.39137" rpy="0 0 0"/>
-    <geometry>
-      <mesh filename="package://urdf_description/meshes/Bar2_1.stl" scale="0.001 0.001 0.001"/>
-    </geometry>
-    <material name="silver"/>
-  </visual>
-  <collision>
-    <origin xyz="-0.122661 0.584079 -0.39137" rpy="0 0 0"/>
-    <geometry>
-      <mesh filename="package://urdf_description/meshes/Bar2_1.stl" scale="0.001 0.001 0.001"/>
-    </geometry>
-  </collision>
-</link>
-<<<<<<< HEAD
-<link name="Bar2_2_sph_x">
-  <inertial>
-  <mass value="0.001"/>
-    <inertia ixx="1e-6" iyy="1e-6" izz="1e-6"
-             ixy="0" iyz="0" ixz="0"/>
-  </inertial>
-</link>
-<link name="Bar2_2_sph_y">
-  <inertial>
-    <mass value="0.001"/>
-    <inertia ixx="1e-6" iyy="1e-6" izz="1e-6"
-             ixy="0" iyz="0" ixz="0"/>
-  </inertial>
-</link>
-<link name="Bar2_2_sph_z">
-  <inertial>
-    <mass value="0.001"/>
-    <inertia ixx="1e-6" iyy="1e-6" izz="1e-6"
-             ixy="0" iyz="0" ixz="0"/>
-  </inertial>
-</link>
-=======
->>>>>>> caddd7ff5a319ac415dbe87685f8ec4c434882f2
-<link name="Wheel1_1">
-  <inertial>
-    <origin xyz="-1.2620295099519119e-06 5.90468842376346e-07 -5.043205407728735e-07" rpy="0 0 0"/>
+<!-- CENTER WHEELS (left and right on center bogie) -->
+<link name="wheel_center_left">
+  <inertial>
+    <origin xyz="0 0 0" rpy="0 0 0"/>
     <mass value="18.64386375159242"/>
     <inertia ixx="0.207999" iyy="0.203936" izz="0.164115" ixy="0.045369" iyz="-0.012432" ixz="-0.013001"/>
   </inertial>
   <visual>
-    <origin xyz="-0.069209 -0.367744 -0.38741" rpy="0 0 0"/>
-    <geometry>
-      <mesh filename="package://urdf_description/meshes/Wheel1_1.stl" scale="0.001 0.001 0.001"/>
-    </geometry>
-    <material name="silver"/>
-  </visual>
-  <collision>
-    <origin xyz="-0.069209 -0.367744 -0.38741" rpy="0 0 0"/>
-    <geometry>
-      <mesh filename="package://urdf_description/meshes/Wheel1_1.stl" scale="0.001 0.001 0.001"/>
-    </geometry>
-  </collision>
-</link>
-<link name="Wheel2_1">
-  <inertial>
-    <origin xyz="-1.1942632050232493e-06 1.057572250023897e-06 1.3665486564562457e-07" rpy="0 0 0"/>
+    <origin xyz="-0.230521 -0.22289 -0.14374" rpy="0 0 0"/>
+    <geometry>
+      <mesh filename="package://urdf_description/meshes/Wheel2_1.stl" scale="0.001 0.001 0.001"/>
+    </geometry>
+    <material name="silver"/>
+  </visual>
+  <collision>
+    <origin xyz="-0.230521 -0.22289 -0.14374" rpy="0 0 0"/>
+    <geometry>
+      <mesh filename="package://urdf_description/meshes/Wheel2_1.stl" scale="0.001 0.001 0.001"/>
+    </geometry>
+  </collision>
+</link>
+<link name="wheel_center_right">
+  <inertial>
+    <origin xyz="0 0 0" rpy="0 0 0"/>
     <mass value="18.64386375159242"/>
     <inertia ixx="0.207999" iyy="0.203936" izz="0.164115" ixy="0.045369" iyz="-0.012432" ixz="-0.013001"/>
   </inertial>
   <visual>
-    <origin xyz="-0.230521 -0.22289 -0.14374" rpy="0 0 0"/>
-    <geometry>
-      <mesh filename="package://urdf_description/meshes/Wheel2_1.stl" scale="0.001 0.001 0.001"/>
-    </geometry>
-    <material name="silver"/>
-  </visual>
-  <collision>
-    <origin xyz="-0.230521 -0.22289 -0.14374" rpy="0 0 0"/>
-    <geometry>
-      <mesh filename="package://urdf_description/meshes/Wheel2_1.stl" scale="0.001 0.001 0.001"/>
-    </geometry>
-  </collision>
-</link>
-<link name="Wheel3_1">
-  <inertial>
-    <origin xyz="-9.592869747443444e-07 3.765590063653512e-07 -1.586157946931177e-07" rpy="0 0 0"/>
-    <mass value="18.64386375159242"/>
-    <inertia ixx="0.207999" iyy="0.203936" izz="0.164115" ixy="0.045369" iyz="-0.012432" ixz="-0.013001"/>
-  </inertial>
-  <visual>
     <origin xyz="-0.143367 -0.225919 0.163611" rpy="0 0 0"/>
     <geometry>
@@ -320,12 +128,34 @@
   </collision>
 </link>
-<link name="Wheel4_1">
-  <inertial>
-    <origin xyz="-3.1802624100851773e-07 -9.095444159501476e-07 -1.648780843410691e-06" rpy="0 0 0"/>
+<!-- REAR ROCKER ARM (Bogie1_1) -->
+<link name="bogie_rear">
+  <inertial>
+    <origin xyz="-0.28590244337464565 0.13764159401794218 -0.3934445335062897" rpy="0 0 0"/>
+    <mass value="2.7421522792728923"/>
+    <inertia ixx="0.028398" iyy="0.027753" izz="0.011564" ixy="-0.004417" iyz="-0.003682" ixz="-0.000457"/>
+  </inertial>
+  <visual>
+    <origin xyz="0.002504 0.454759 -0.288737" rpy="0 0 0"/>
+    <geometry>
+      <mesh filename="package://urdf_description/meshes/Bogie1_1.stl" scale="0.001 0.001 0.001"/>
+    </geometry>
+    <material name="silver"/>
+  </visual>
+  <collision>
+    <origin xyz="0.002504 0.454759 -0.288737" rpy="0 0 0"/>
+    <geometry>
+      <mesh filename="package://urdf_description/meshes/Bogie1_1.stl" scale="0.001 0.001 0.001"/>
+    </geometry>
+  </collision>
+</link>
+<!-- REAR WHEEL (on Rear Rocker) -->
+<link name="wheel_rear">
+  <inertial>
+    <origin xyz="0 0 0" rpy="0 0 0"/>
     <mass value="18.64386375159242"/>
     <inertia ixx="0.207997" iyy="0.203937" izz="0.164114" ixy="0.04537" iyz="-0.012432" ixz="-0.013"/>
   </inertial>
   <visual>
-    <origin xyz="0.291017 0.34301 0.210668" rpy="0 0 0"/>
+    <origin xyz="-0.288513 0.111749 -0.499405" rpy="0 0 0"/>
     <geometry>
       <mesh filename="package://urdf_description/meshes/Wheel4_1.stl" scale="0.001 0.001 0.001"/>
@@ -334,5 +164,5 @@
   </visual>
   <collision>
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